Commit message: add entity node to subscribe on robot_description topic

File: youbot/youbot_model_description/urdf/youbot_base.xacro (robot description, xacro)
@@ -44,5 +44,5 @@
     </link>
     <joint name="base_footprint_joint" type="fixed">
-      <origin rpy="0 0 0" xyz="0 0 0"/>
+      <origin rpy="0 0 0" xyz="0 0 0.0841"/>
       <child link="base_link"/>
       <parent link="base_footprint"/>
