Commit message: install plugin for lidar

File: youbot/youbot_controller/src/youbot_lidar_gazebo_plugins.urdf.xacro (robot description, xacro)
@@ -2,9 +2,8 @@
 <robot xmlns:xacro="http://www.ros.org/wiki/xacro" >
   <gazebo reference="base_laser_front_link">
-    <sensor name='base_laser_front' type='ray'>
-      <pose relative_to="lidar_frame">0 0 0 0 0 0</pose>
+    <sensor name='base_laser_front' type='gpu_lidar'>
+      <pose>0 0 0 0 0 0</pose>
       <visualize>true</visualize>
       <update_rate>10</update_rate>
-      <topic>lidar</topic>
       <ray>
         <scan>
@@ -23,6 +22,6 @@
         </scan>
           <range>
-              <min>0.05</min>
-              <max>5.6</max>
+              <min>0.3</min>
+              <max>5.4</max>
               <resolution>0.36</resolution>
           </range>
@@ -35,6 +34,8 @@
       <always_on>1</always_on>
     </sensor>
-    <plugin name='gazebo_ros_base_laser_front_controller' filename='gz-sim-sensors-system'>
-      <render_engine>ogre2</render_engine>
+    <plugin name='gazebo_ros_base_laser_front_controller' filename='libgazebo_ros_gpu_laser.so'>
+      <frame_name>laser_front_link</frame_name>
+      <output_typ>sensor_msgs/LaserScan</output_typ>
+      <topic>/scan</topic>
     </plugin>
   </gazebo>

File: youbot/youbot_model_description/urdf/youbot.urdf.xacro (robot description, xacro)
@@ -2,11 +2,11 @@
 <robot xmlns:xacro="http://www.ros.org/wiki/xacro" name="youbot">
     <xacro:include filename="youbot_base.xacro" />
+    <xacro:include filename="youbot_lidar.xacro"/>
+    <xacro:include filename="$(find youbot_controller)/src/youbot_lidar_gazebo_plugins.urdf.xacro"/>
     <xacro:include filename="$(find youbot_controller)/src/youbot_base_gazebo_plugins.urdf.xacro"/>
     <!--
     <xacro:include filename="$(find youbot_controller)/src/youbot_arm_gazebo_plugins.urdf.xacro"/>
       <xacro:include filename="$(find youbot_controller)/src/ros_controller.urdf.xacro"/>
-   <xacro:include filename="youbot_lidar.xacro"/>
-    <xacro:include filename="$(find youbot_controller)/src/youbot_lidar_gazebo_plugins.urdf.xacro"/>
-     <xacro:include filename="youbot_arm.xacro" />
+   <xacro:include filename="youbot_arm.xacro" />
     -->
 </robot>

File: youbot/youbot_model_description/urdf/youbot_lidar.xacro (robot description, xacro)
@@ -7,5 +7,5 @@
         <child link="base_laser_front_link"/>
     </joint>
-    <link name="base_laser_front_link" type="gpu_lidar">
+    <link name="base_laser_front_link" >
         <inertial>
           <mass value="0.16"/>
