Commit message: start with lidar

File: youbot/youbot_controller/src/youbot_base_gazebo_plugins.urdf.xacro (robot description, xacro)
@@ -5,11 +5,66 @@
         <left_joint>wheel_joint_fl</left_joint>
         <left_joint>wheel_joint_bl</left_joint>
+        <left_joint>caster_joint_fl</left_joint>
+        <left_joint>caster_joint_bl</left_joint>
         <right_joint>wheel_joint_fr</right_joint>
         <right_joint>wheel_joint_br</right_joint>
+        <right_joint>caster_joint_fr</right_joint>
+        <right_joint>caster_joint_br</right_joint>
+        <wheel_separation>0.3</wheel_separation>
+        <wheel_diameter>0.0475</wheel_diameter>
+        <odom_publish_frequency>10</odom_publish_frequency>
+        <topic>cmd_vel</topic>
+        <robot_base_frame>base_footprint</robot_base_frame>
+        <odometry_frame>odom</odometry_frame>
+        <publish_odom>true</publish_odom>
+        <publish_odom_tf>true</publish_odom_tf>
+        <publish_wheel_tf>true</publish_wheel_tf>
+      </plugin>
+      <!--
+        <plugin name='base_controller'
+              filename='libgazebo_ros_planar_move.so'>
+          <update_rate>100</update_rate>
+          <publish_rate>10</publish_rate>
+          <publish_odom>true</publish_odom>
+          <publish_odom_tf>true</publish_odom_tf>
+          <robot_base_frame>base_footprint</robot_base_frame>
+          <covariance_x>0.0001</covariance_x>
+          <covariance_y>0.0001</covariance_y>
+          <covariance_yaw>0.01</covariance_yaw>
+        </plugin>
+      <gazebo reference="wheel_link_fl">
+        <mu1 value="0.001"/>
+        <mu2 value ="0.001"/>
+      </gazebo>
+      <gazebo reference="wheel_link_fr">
+        <mu1 value="0.001"/>
+        <mu2 value ="0.001"/>
+      </gazebo>
+      <gazebo reference="wheel_link_bl">
+        <mu1 value="0.001"/>
+        <mu2 value ="0.001"/>
+      </gazebo>
+      <gazebo reference="wheel_link_br">
+        <mu1 value="0.001"/>
+        <mu2 value ="0.001"/>
+      </gazebo>
+      <plugin name="omni_steering" filename="libgazebo_ros_planar_move.so">
+        <commandTopic>cmd_vel</commandTopic>
+        <odometryTopic>odom</odometryTopic>
+        <odometryRate>10</odometryRate>
+        <robotBaseFrame>base_footprint</robotBaseFrame>
+        <publishTF>true</publishTF>
+      </plugin>
+    <plugin name="skid_steer_drive_controller" filename="libgazebo_ros_skid_steer_drive.so">
+        <topic>cmd_vel</topic>
+        <publishRate>10</publishRate>
+        <frontLeftJoint>wheel_joint_fl</frontLeftJoint>
+        <frontRightJoint>wheel_joint_fr</frontRightJoint>
+        <rearLeftJoint>wheel_joint_bl</rearLeftJoint>
+        <rearRightJoint>wheel_joint_br</rearRightJoint>
         <wheel_separation>0.316</wheel_separation>
         <wheel_radius>0.3</wheel_radius>
-        <odom_publish_frequency>1</odom_publish_frequency>
-        <topic>cmd_vel</topic>
       </plugin>
+  -->
     </gazebo>
     <gazebo>
@@ -24,5 +79,5 @@
       <plugin name="ignition::gazebo::systems::JointStatePublisher"
         filename="ignition-gazebo-joint-state-publisher-system">
-        <update_rate>100</update_rate>
+        <update_rate>10</update_rate>
         <joint_name>wheel_joint_bl</joint_name>
         <joint_name>wheel_joint_br</joint_name>

File: youbot/youbot_controller/src/youbot_lidar_gazebo_plugins.urdf.xacro (robot description, xacro)
@@ -1,11 +1,44 @@
 <?xml version="1.0"?>
 <robot xmlns:xacro="http://www.ros.org/wiki/xacro" >
-<plugin name='gazebo_ros_base_laser_front_controller'
-                          filename='libgazebo_ros_ray_sensor.so'>
-              <ros>
-                <namespace>/youbot</namespace>
-                <argument>--ros-args --remap ~/out:=scan</argument>
-              </ros>
-              <output_type>sensor_msgs/LaserScan</output_type>
-            </plugin>
+  <gazebo reference="base_laser_front_link">
+    <sensor name='base_laser_front' type='gpu_lidar'>
+      <pose>0 0 0 0 0 0</pose>
+      <update_rate>10</update_rate>
+      <visualize>true</visualize>
+      <ray>
+        <scan>
+          <horizontal>
+              <samples>150</samples>
+              <resolution>1</resolution>
+              <min_angle>-1.57</min_angle>
+              <max_angle>1.57</max_angle>
+          </horizontal>
+          <vertical>
+              <samples>1</samples>
+              <min_angle>0</min_angle>
+              <max_angle>0</max_angle>
+          </vertical>
+        </scan>
+          <range>
+              <min>0.05</min>
+              <max>5.6</max>
+              <resolution>0.36</resolution>
+          </range>
+          <noise>
+              <type>gaussian</type>
+              <mean>0.00</mean>
+              <stddev>0.01</stddev>
+          </noise>
+      </ray>
+    </sensor>
+    <plugin name='gazebo_ros_base_laser_front_controller' filename='libignition-gazebo-sensors-system.so'>
+      <ros>
+       <!--   <argument> -  -ros-args - -remap ~/out:=scan</argument>
+      -->
+      <argument>~/out:=scan</argument>
+      </ros>
+      <output_type>sensor_msgs/LaserScan</output_type>
+      <frame_name>/scan</frame_name>
+    </plugin>
+  </gazebo>
 </robot>

File: youbot/youbot_model_description/urdf/youbot.urdf.xacro (robot description, xacro)
@@ -4,8 +4,8 @@
     <xacro:include filename="youbot_lidar.xacro" />
     <xacro:include filename="$(find youbot_controller)/src/youbot_base_gazebo_plugins.urdf.xacro"/>
+    <xacro:include filename="$(find youbot_controller)/src/youbot_lidar_gazebo_plugins.urdf.xacro"/>
     <!--
     <xacro:include filename="$(find youbot_controller)/src/youbot_arm_gazebo_plugins.urdf.xacro"/>
       <xacro:include filename="$(find youbot_controller)/src/ros_controller.urdf.xacro"/>
-    <xacro:include filename="$(find youbot_controller)/src/youbot_lidar_gazebo_plugins.urdf.xacro"/>
      <xacro:include filename="youbot_arm.xacro" />
     -->

File: youbot/youbot_model_description/urdf/youbot_base.xacro (robot description, xacro)
@@ -44,5 +44,5 @@
     </link>
     <joint name="base_footprint_joint" type="fixed">
-      <origin rpy="0 0 0" xyz="0 0 0.0841"/>
+      <origin rpy="0 0 0" xyz="0 0 0"/>
       <child link="base_link"/>
       <parent link="base_footprint"/>
@@ -56,5 +56,5 @@
       </inertial>
       <visual>
-        <origin rpy="0 0 0" xyz="0 0 0"/>
+        <origin rpy="0 0 0" xyz="0 0 0.0841"/>
         <geometry>
           <mesh filename="package://youbot_model_description/urdf/meshes/youbot_base/base.dae"/>
@@ -62,5 +62,5 @@
       </visual>
       <collision>
-        <origin rpy="0 0 0" xyz="0 0 0"/>
+        <origin rpy="0 0 0" xyz="0 0 0.0841"/>
         <geometry>
           <mesh filename="package://youbot_model_description/urdf/meshes/youbot_base/base_convex.dae"/>
@@ -69,8 +69,9 @@
     </link>
     <joint name="caster_joint_fl" type="fixed">
-      <origin rpy="0 0 0" xyz="0.228 0.158 -0.034"/>
+      <origin rpy="0 0 0" xyz="0.228 0.158 0.0501"/>
       <axis xyz="0 0 1"/>
       <parent link="base_link"/>
       <child link="caster_link_fl"/>
+      <limit effort="10" velocity="100"/>
     </joint>
     <link name="caster_link_fl">
@@ -85,7 +86,7 @@
       <axis xyz="0 1 0"/>
       <limit effort="30" velocity="10"/>
+      <dynamics damping="1.0" friction="1.0"/>
       <origin rpy="0 0 0" xyz="0.0 0.0 0.0"/>
       <parent link="caster_link_fl"/>
-      <dynamics damping="1.0" friction="1.0"/>
       <child link="wheel_link_fl"/>
     </joint>
@@ -110,8 +111,9 @@
     </link>
     <joint name="caster_joint_fr" type="fixed">
-      <origin rpy="0 0 0" xyz="0.228 -0.158 -0.034"/>
+      <origin rpy="0 0 0" xyz="0.228 -0.158 0.0501"/>
       <axis xyz="0 0 1"/>
       <parent link="base_link"/>
       <child link="caster_link_fr"/>
+      <limit effort="10" velocity="100"/>
     </joint>
     <link name="caster_link_fr">
@@ -151,8 +153,9 @@
     </link>
     <joint name="caster_joint_bl" type="fixed">
-      <origin rpy="0 0 0" xyz="-0.228 0.158 -0.034"/>
+      <origin rpy="0 0 0" xyz="-0.228 0.158 0.0501"/>
       <axis xyz="0 0 1"/>
       <parent link="base_link"/>
       <child link="caster_link_bl"/>
+      <limit effort="10" velocity="100"/>
     </joint>
     <link name="caster_link_bl">
@@ -166,5 +169,4 @@
     <joint name="wheel_joint_bl" type="continuous">
       <axis xyz="0 1 0"/>
-      <limit effort="10" velocity="10"/>
       <limit effort="30" velocity="10"/>
       <dynamics damping="1.0" friction="1.0"/>
@@ -193,8 +195,9 @@
     </link>
     <joint name="caster_joint_br" type="fixed">
-      <origin rpy="0 0 0" xyz="-0.228 -0.158 -0.034"/>
+      <origin rpy="0 0 0" xyz="-0.228 -0.158 0.0501"/>
       <axis xyz="0 0 1"/>
       <parent link="base_link"/>
       <child link="caster_link_br"/>
+      <limit effort="10" velocity="100"/>
     </joint>
     <link name="caster_link_br">

File: youbot/youbot_model_description/urdf/youbot_lidar.xacro (robot description, xacro)
@@ -3,9 +3,9 @@
     <joint name="base_laser_front_hokuyo_urg04_laser_joint" type="fixed">
         <axis xyz="0 1 0"/>
-        <origin rpy="3.14159 3.14159 3.14159" xyz="0.3 0 -0.03"/>
+        <origin rpy="3.14159 3.14159 3.14159" xyz="0.3 0 0.051"/>
         <parent link="base_link"/>
         <child link="base_laser_front_link"/>
     </joint>
-    <link name="base_laser_front_link" type="laser">
+    <link name="base_laser_front_link" type="gpu_lidar">
         <inertial>
           <mass value="0.16"/>
@@ -25,37 +25,4 @@
           </geometry>
         </collision>
-        <sensor name='base_laser_front'
-                        type='gpu_ray'>
-                    <always_on>1</always_on>
-                    <update_rate>10</update_rate>
-                    <visualize>0</visualize>
-                    <ray>
-                        <scan>
-                            <horizontal>
-                                <samples>150</samples>
-                                <resolution>1</resolution>
-                                <min_angle>-1.57</min_angle>
-                                <max_angle>1.57</max_angle>
-                            </horizontal>
-                            <vertical>
-                                <samples>1</samples>
-                                <min_angle>0</min_angle>
-                                <max_angle>0</max_angle>
-                            </vertical>
-                        </scan>
-                        <range>
-                            <min>0.05</min>
-                            <max>5.6</max>
-                            <resolution>0.36</resolution>
-                        </range>
-                        <noise>
-                            <type>gaussian</type>
-                            <mean>0.00</mean>
-                            <stddev>0.01</stddev>
-                        </noise>
-                    </ray>
-                    <update_rate>10</update_rate>
-                    <pose frame=''>0.3 0 -0.03 0 -0 0</pose>
-                </sensor>
     </link>
 </robot>
