Commit message: init

File: youbot/youbot_controller/src/youbot_base_gazebo_plugins.urdf.xacro (robot description, xacro)
@@ -2,17 +2,13 @@
 <robot xmlns:xacro="http://www.ros.org/wiki/xacro" >
     <gazebo>
-      <plugin filename="libignition-gazebo-diff-drive-system.so" name="ignition::gazebo::systems::DiffDrive">
-        <left_joint>wheel_joint_fl</left_joint>
+      <plugin filename="libgazebo_ros_diff_drive.so" name="DiffDrive">
+     <!--  <plugin filename="gz-sim-diff-drive-system" name="DiffDrive">-->
+        <left_joint_1>wheel_joint_fl</left_joint_1>
         <left_joint>wheel_joint_bl</left_joint>
-        <left_joint>caster_joint_fl</left_joint>
-        <left_joint>caster_joint_bl</left_joint>
-        <right_joint>wheel_joint_fr</right_joint>
+        <right_joint_1>wheel_joint_fr</right_joint_1>
         <right_joint>wheel_joint_br</right_joint>
-        <right_joint>caster_joint_fr</right_joint>
-        <right_joint>caster_joint_br</right_joint>
         <wheel_separation>0.3</wheel_separation>
         <wheel_diameter>0.0475</wheel_diameter>
         <odom_publish_frequency>10</odom_publish_frequency>
-        <topic>cmd_vel</topic>
         <robot_base_frame>base_footprint</robot_base_frame>
         <odometry_frame>odom</odometry_frame>
@@ -21,11 +17,13 @@
         <publish_wheel_tf>true</publish_wheel_tf>
       </plugin>
-      <!--
-        <plugin name='base_controller'
+        <plugin name='planar_move'
               filename='libgazebo_ros_planar_move.so'>
-          <update_rate>100</update_rate>
+         <topic>cmd_vel</topic>
+          <update_rate>10</update_rate>
           <publish_rate>10</publish_rate>
           <publish_odom>true</publish_odom>
           <publish_odom_tf>true</publish_odom_tf>
+          <odometyTopic>odom</odometyTopic>
+          <odometryFrame>odom</odometryFrame>
           <robot_base_frame>base_footprint</robot_base_frame>
           <covariance_x>0.0001</covariance_x>
@@ -33,4 +31,16 @@
           <covariance_yaw>0.01</covariance_yaw>
         </plugin>
+      </gazebo>
+<!--
+      <gazebo>
+        <plugin name="gazebo-ros-joint-state-publisher-base"
+                filename="libgazebo-ros-joint-state-publisher.so">
+          <update_rate>10</update_rate>
+          <joint_name>wheel_joint_bl</joint_name>
+          <joint_name>wheel_joint_br</joint_name>
+          <joint_name>wheel_joint_fl</joint_name>
+          <joint_name>wheel_joint_fr</joint_name>
+        </plugin>
+      </gazebo>
       <gazebo reference="wheel_link_fl">
         <mu1 value="0.001"/>
@@ -67,5 +77,5 @@
       </plugin>
   -->
-    </gazebo>
+      <!--
     <gazebo>
       <plugin
@@ -94,18 +104,4 @@
       </plugin>
     </gazebo>
-   <!--
-     <gazebo>
-      <plugin name="gazebo-ros-joint-state-publisher-base"
-              filename="libgazebo-ros-joint-state-publisher.so">
-        <ros>
-          <namespace>/youbot</namespace>
-        </ros>
-        <update_rate>100</update_rate>
-        <joint_name>wheel_joint_bl</joint_name>
-        <joint_name>wheel_joint_br</joint_name>
-        <joint_name>wheel_joint_fl</joint_name>
-        <joint_name>wheel_joint_fr</joint_name>
-      </plugin>
-    </gazebo>
       -->
 </robot>

File: youbot/youbot_controller/src/youbot_lidar_gazebo_plugins.urdf.xacro (robot description, xacro)
@@ -2,42 +2,6 @@
 <robot xmlns:xacro="http://www.ros.org/wiki/xacro" >
   <gazebo reference="base_laser_front_link">
-    <sensor name='base_laser_front' type='gpu_lidar'>
-      <pose>0 0 0 0 0 0</pose>
-      <update_rate>10</update_rate>
-      <visualize>true</visualize>
-      <ray>
-        <scan>
-          <horizontal>
-              <samples>150</samples>
-              <resolution>1</resolution>
-              <min_angle>-1.57</min_angle>
-              <max_angle>1.57</max_angle>
-          </horizontal>
-          <vertical>
-              <samples>1</samples>
-              <min_angle>0</min_angle>
-              <max_angle>0</max_angle>
-          </vertical>
-        </scan>
-          <range>
-              <min>0.05</min>
-              <max>5.6</max>
-              <resolution>0.36</resolution>
-          </range>
-          <noise>
-              <type>gaussian</type>
-              <mean>0.00</mean>
-              <stddev>0.01</stddev>
-          </noise>
-      </ray>
-    </sensor>
-    <plugin name='gazebo_ros_base_laser_front_controller' filename='libignition-gazebo-sensors-system.so'>
-      <ros>
-       <!--   <argument> -  -ros-args - -remap ~/out:=scan</argument>
-      -->
-      <argument>~/out:=scan</argument>
-      </ros>
-      <output_type>sensor_msgs/LaserScan</output_type>
-      <frame_name>/scan</frame_name>
+    <plugin name='gazebo_ros_base_laser_front_controller' filename='gz-sim-sensors-system'>
+      <render_engine>ogre2</render_engine>
     </plugin>
   </gazebo>

File: youbot/youbot_model_description/urdf/youbot.urdf.xacro (robot description, xacro)
@@ -2,7 +2,7 @@
 <robot xmlns:xacro="http://www.ros.org/wiki/xacro" name="youbot">
     <xacro:include filename="youbot_base.xacro" />
+    <xacro:include filename="$(find youbot_controller)/src/youbot_lidar_gazebo_plugins.urdf.xacro"/>
     <xacro:include filename="youbot_lidar.xacro" />
     <xacro:include filename="$(find youbot_controller)/src/youbot_base_gazebo_plugins.urdf.xacro"/>
-    <xacro:include filename="$(find youbot_controller)/src/youbot_lidar_gazebo_plugins.urdf.xacro"/>
     <!--
     <xacro:include filename="$(find youbot_controller)/src/youbot_arm_gazebo_plugins.urdf.xacro"/>

File: youbot/youbot_model_description/urdf/youbot_base.xacro (robot description, xacro)
@@ -48,15 +48,15 @@
       <parent link="base_footprint"/>
     </joint>
-    <!-- BASE_LINK-->
+   <!--  BASE_LINK-->
     <link name="base_link">
       <inertial>
-        <mass value="22.0"/>
-        <origin xyz="0 0 0"/>
-        <inertia ixx="5.652232699207" ixy="-0.009719934438" ixz="1.293988226423" iyy="5.669473158652" iyz="-0.007379583694" izz="3.683196351726"/>
+        <mass value="19.0"/>
+        <origin xyz="0 0 0"/>
+        <inertia ixx="5.652232699207" ixy="0" ixz="1.293988226423" iyy="5.669473158652" iyz="0" izz="3.683196351726"/>
       </inertial>
       <visual>
         <origin rpy="0 0 0" xyz="0 0 0.0841"/>
         <geometry>
-          <mesh filename="package://youbot_model_description/urdf/meshes/youbot_base/base.dae"/>
+          <mesh filename="$(find youbot_model_description)/urdf/meshes/youbot_base/base.dae"/>
         </geometry>
       </visual>
@@ -64,5 +64,5 @@
         <origin rpy="0 0 0" xyz="0 0 0.0841"/>
         <geometry>
-          <mesh filename="package://youbot_model_description/urdf/meshes/youbot_base/base_convex.dae"/>
+          <mesh filename="$(find youbot_model_description)/urdf/meshes/youbot_base/base_convex.dae"/>
         </geometry>
       </collision>
@@ -79,5 +79,5 @@
         <mass value="0.1"/>
         <origin xyz="0 0 0"/>
-        <inertia ixx="0.012411765597" ixy="-0.000711733678" ixz="0.00050272983" iyy="0.015218160428" iyz="-0.000004273467" izz="0.011763977943"/>
+        <inertia ixx="0.012411765597" ixy="0" ixz="0.00050272983" iyy="0.015218160428" iyz="0" izz="0.011763977943"/>
       </inertial>
     </link>
@@ -93,12 +93,12 @@
     <link name="wheel_link_fl">
       <inertial>
-        <mass value="0.4"/>
-        <origin xyz="0 0 0"/>
-        <inertia ixx="0.012411765597" ixy="-0.000711733678" ixz="0.00050272983" iyy="0.015218160428" iyz="-0.000004273467" izz="0.011763977943"/>
-      </inertial>
-      <visual>
-        <origin rpy="0 0 0" xyz="0 0 0"/>
-        <geometry>
-          <mesh filename="package://youbot_model_description/urdf/meshes/youbot_base/front-left_wheel.dae"/>
+        <mass value="1.4"/>
+        <origin xyz="0 0 0"/>
+        <inertia ixx="0.012411765597" ixy="0" ixz="0.00050272983" iyy="0.015218160428" iyz="0" izz="0.011763977943"/>
+      </inertial>
+      <visual>
+        <origin rpy="0 0 0" xyz="0 0 0"/>
+        <geometry>
+          <mesh filename="$(find youbot_model_description)/urdf/meshes/youbot_base/front-left_wheel.dae"/>
         </geometry>
       </visual>
@@ -121,5 +121,5 @@
         <mass value="0.1"/>
         <origin xyz="0 0 0"/>
-        <inertia ixx="0.012411765597" ixy="-0.000711733678" ixz="0.00050272983" iyy="0.015218160428" iyz="-0.000004273467" izz="0.011763977943"/>
+        <inertia ixx="0.012411765597" ixy="0" ixz="0.00050272983" iyy="0.015218160428" iyz="0" izz="0.011763977943"/>
       </inertial>
     </link>
@@ -135,12 +135,12 @@
     <link name="wheel_link_fr">
       <inertial>
-        <mass value="0.4"/>
-        <origin xyz="0 0 0"/>
-        <inertia ixx="0.012411765597" ixy="-0.000711733678" ixz="0.00050272983" iyy="0.015218160428" iyz="-0.000004273467" izz="0.011763977943"/>
-      </inertial>
-      <visual>
-        <origin rpy="0 0 0" xyz="0 0 0"/>
-        <geometry>
-          <mesh filename="package://youbot_model_description/urdf/meshes/youbot_base/front-right_wheel.dae"/>
+        <mass value="1.4"/>
+        <origin xyz="0 0 0"/>
+        <inertia ixx="0.012411765597" ixy="0" ixz="0.00050272983" iyy="0.015218160428" iyz="0" izz="0.011763977943"/>
+      </inertial>
+      <visual>
+        <origin rpy="0 0 0" xyz="0 0 0"/>
+        <geometry>
+          <mesh filename= "$(find youbot_model_description)/urdf/meshes/youbot_base/front-right_wheel.dae"/>
         </geometry>
       </visual>
@@ -163,5 +163,5 @@
         <mass value="0.1"/>
         <origin xyz="0 0 0"/>
-        <inertia ixx="0.012411765597" ixy="-0.000711733678" ixz="0.00050272983" iyy="0.015218160428" iyz="-0.000004273467" izz="0.011763977943"/>
+        <inertia ixx="0.012411765597" ixy="0.000711733678" ixz="0.00050272983" iyy="0.015218160428" iyz="0.000004273467" izz="0.011763977943"/>
       </inertial>
     </link>
@@ -177,12 +177,12 @@
     <link name="wheel_link_bl">
       <inertial>
-        <mass value="0.4"/>
-        <origin xyz="0 0 0"/>
-        <inertia ixx="0.012411765597" ixy="-0.000711733678" ixz="0.00050272983" iyy="0.015218160428" iyz="-0.000004273467" izz="0.011763977943"/>
-      </inertial>
-      <visual>
-        <origin rpy="0 0 0" xyz="0 0 0"/>
-        <geometry>
-          <mesh filename="package://youbot_model_description/urdf/meshes/youbot_base/back-left_wheel.dae"/>
+        <mass value="1.4"/>
+        <origin xyz="0 0 0"/>
+        <inertia ixx="0.012411765597" ixy="0.000711733678" ixz="0.00050272983" iyy="0.015218160428" iyz="0.000004273467" izz="0.011763977943"/>
+      </inertial>
+      <visual>
+        <origin rpy="0 0 0" xyz="0 0 0"/>
+        <geometry>
+          <mesh filename="$(find youbot_model_description)/urdf/meshes/youbot_base/back-left_wheel.dae"/>
         </geometry>
       </visual>
@@ -205,5 +205,5 @@
         <mass value="0.1"/>
         <origin xyz="0 0 0"/>
-        <inertia ixx="0.012411765597" ixy="-0.000711733678" ixz="0.00050272983" iyy="0.015218160428" iyz="-0.000004273467" izz="0.011763977943"/>
+        <inertia ixx="0.012411765597" ixy="0.000711733678" ixz="0.00050272983" iyy="0.015218160428" iyz="0.000004273467" izz="0.011763977943"/>
       </inertial>
     </link>
@@ -219,12 +219,12 @@
     <link name="wheel_link_br">
       <inertial>
-        <mass value="0.4"/>
-        <origin xyz="0 0 0"/>
-        <inertia ixx="0.012411765597" ixy="-0.000711733678" ixz="0.00050272983" iyy="0.015218160428" iyz="-0.000004273467" izz="0.011763977943"/>
-      </inertial>
-      <visual>
-        <origin rpy="0 0 0" xyz="0 0 0"/>
-        <geometry>
-          <mesh filename="package://youbot_model_description/urdf/meshes/youbot_base/back-right_wheel.dae"/>
+        <mass value="1.4"/>
+        <origin xyz="0 0 0"/>
+        <inertia ixx="0.012411765597" ixy="0.000711733678" ixz="0.00050272983" iyy="0.015218160428" iyz="0.000004273467" izz="0.011763977943"/>
+      </inertial>
+      <visual>
+        <origin rpy="0 0 0" xyz="0 0 0"/>
+        <geometry>
+          <mesh filename="$(find youbot_model_description)/urdf/meshes/youbot_base/back-right_wheel.dae"/>
         </geometry>
       </visual>

File: youbot/youbot_model_description/urdf/youbot_lidar.xacro (robot description, xacro)
@@ -7,4 +7,7 @@
         <child link="base_laser_front_link"/>
     </joint>
+  <frame name="lidar_frame" attached_to="base_laser_front_link">
+    <pose>0 0 0 0 0 0</pose>
+  </frame>
     <link name="base_laser_front_link" type="gpu_lidar">
         <inertial>
@@ -16,5 +19,5 @@
           <origin rpy="0 0 0" xyz="0 0 0"/>
           <geometry>
-            <mesh filename="package://youbot_model_description/urdf/meshes/sensors/hokuyo.dae"/>
+            <mesh filename="$(find youbot_model_description)/urdf/meshes/sensors/hokuyo.dae"/>
           </geometry>
         </visual>
@@ -22,7 +25,40 @@
           <origin rpy="0 0 0" xyz="0 0 0"/>
           <geometry>
-            <mesh filename="package://youbot_model_description/urdf/meshes/sensors/hokuyo_convex.dae"/>
+            <mesh filename="$(find youbot_model_description)/urdf/meshes/sensors/hokuyo_convex.dae"/>
           </geometry>
         </collision>
+        <sensor name='base_laser_front' type='gpu_lidar'>
+          <pose relative_to="lidar_frame">0 0 0 0 0 0</pose>
+          <update_rate>10</update_rate>
+          <topic>lidar</topic>
+          <ray>
+            <scan>
+              <horizontal>
+                  <samples>150</samples>
+                  <resolution>1</resolution>
+                  <min_angle>-1.57</min_angle>
+                  <max_angle>1.57</max_angle>
+              </horizontal>
+             <vertical>
+                  <samples>1</samples>
+                  <resolution>0.01</resolution>
+                  <min_angle>0</min_angle>
+                  <max_angle>0</max_angle>
+              </vertical>
+            </scan>
+              <range>
+                  <min>0.05</min>
+                  <max>5.6</max>
+                  <resolution>0.36</resolution>
+              </range>
+             <!-- <noise>
+                  <type>gaussian</type>
+                  <mean>0.00</mean>
+                  <stddev>0.01</stddev>
+              </noise>-->
+          </ray>
+          <always_on>1</always_on>
+          <visualize>true</visualize>
+        </sensor>
     </link>
 </robot>

Commit message: lidar

File: youbot/youbot_controller/src/youbot_base_gazebo_plugins.urdf.xacro (robot description, xacro)
@@ -59,21 +59,4 @@
         <mu2 value ="0.001"/>
       </gazebo>
-      <plugin name="omni_steering" filename="libgazebo_ros_planar_move.so">
-        <commandTopic>cmd_vel</commandTopic>
-        <odometryTopic>odom</odometryTopic>
-        <odometryRate>10</odometryRate>
-        <robotBaseFrame>base_footprint</robotBaseFrame>
-        <publishTF>true</publishTF>
-      </plugin>
-    <plugin name="skid_steer_drive_controller" filename="libgazebo_ros_skid_steer_drive.so">
-        <topic>cmd_vel</topic>
-        <publishRate>10</publishRate>
-        <frontLeftJoint>wheel_joint_fl</frontLeftJoint>
-        <frontRightJoint>wheel_joint_fr</frontRightJoint>
-        <rearLeftJoint>wheel_joint_bl</rearLeftJoint>
-        <rearRightJoint>wheel_joint_br</rearRightJoint>
-        <wheel_separation>0.316</wheel_separation>
-        <wheel_radius>0.3</wheel_radius>
-      </plugin>
   -->
       <!--
@@ -86,22 +69,4 @@
          </plugin>
     </gazebo>
-    <gazebo>
-      <plugin name="ignition::gazebo::systems::JointStatePublisher"
-        filename="ignition-gazebo-joint-state-publisher-system">
-        <update_rate>10</update_rate>
-        <joint_name>wheel_joint_bl</joint_name>
-        <joint_name>wheel_joint_br</joint_name>
-        <joint_name>wheel_joint_fl</joint_name>
-        <joint_name>wheel_joint_fr</joint_name>
-      </plugin>
-    </gazebo>
-    <gazebo>
-      <plugin filename="ignition-gazebo-pose-publisher-system" name="ignition::gazebo::systems::PosePublisher">
-        <publish_link_pose>true</publish_link_pose>
-        <use_pose_vector_msg>true</use_pose_vector_msg>
-        <static_publisher>true</static_publisher>
-        <static_update_frequency>1</static_update_frequency>
-      </plugin>
-    </gazebo>
       -->
 </robot>

File: youbot/youbot_controller/src/youbot_lidar_gazebo_plugins.urdf.xacro (robot description, xacro)
@@ -2,4 +2,37 @@
 <robot xmlns:xacro="http://www.ros.org/wiki/xacro" >
   <gazebo reference="base_laser_front_link">
+    <sensor name='base_laser_front' type='ray'>
+      <pose relative_to="lidar_frame">0 0 0 0 0 0</pose>
+      <visualize>true</visualize>
+      <update_rate>10</update_rate>
+      <topic>lidar</topic>
+      <ray>
+        <scan>
+          <horizontal>
+              <samples>150</samples>
+              <resolution>1</resolution>
+              <min_angle>-1.57</min_angle>
+              <max_angle>1.57</max_angle>
+          </horizontal>
+         <vertical>
+              <samples>1</samples>
+              <resolution>0.01</resolution>
+              <min_angle>0</min_angle>
+              <max_angle>0</max_angle>
+          </vertical>
+        </scan>
+          <range>
+              <min>0.05</min>
+              <max>5.6</max>
+              <resolution>0.36</resolution>
+          </range>
+         <!-- <noise>
+              <type>gaussian</type>
+              <mean>0.00</mean>
+              <stddev>0.01</stddev>
+          </noise>-->
+      </ray>
+      <always_on>1</always_on>
+    </sensor>
     <plugin name='gazebo_ros_base_laser_front_controller' filename='gz-sim-sensors-system'>
       <render_engine>ogre2</render_engine>

File: youbot/youbot_model_description/urdf/youbot.urdf.xacro (robot description, xacro)
@@ -2,10 +2,10 @@
 <robot xmlns:xacro="http://www.ros.org/wiki/xacro" name="youbot">
     <xacro:include filename="youbot_base.xacro" />
-    <xacro:include filename="$(find youbot_controller)/src/youbot_lidar_gazebo_plugins.urdf.xacro"/>
-    <xacro:include filename="youbot_lidar.xacro" />
     <xacro:include filename="$(find youbot_controller)/src/youbot_base_gazebo_plugins.urdf.xacro"/>
     <!--
     <xacro:include filename="$(find youbot_controller)/src/youbot_arm_gazebo_plugins.urdf.xacro"/>
       <xacro:include filename="$(find youbot_controller)/src/ros_controller.urdf.xacro"/>
+   <xacro:include filename="youbot_lidar.xacro"/>
+    <xacro:include filename="$(find youbot_controller)/src/youbot_lidar_gazebo_plugins.urdf.xacro"/>
      <xacro:include filename="youbot_arm.xacro" />
     -->

File: youbot/youbot_model_description/urdf/youbot_base.xacro (robot description, xacro)
@@ -59,5 +59,5 @@
         <geometry>
           <mesh filename="$(find youbot_model_description)/urdf/meshes/youbot_base/base.dae"/>
-        </geometry>
+      </geometry>
       </visual>
       <collision>

File: youbot/youbot_model_description/urdf/youbot_lidar.xacro (robot description, xacro)
@@ -7,7 +7,4 @@
         <child link="base_laser_front_link"/>
     </joint>
-  <frame name="lidar_frame" attached_to="base_laser_front_link">
-    <pose>0 0 0 0 0 0</pose>
-  </frame>
     <link name="base_laser_front_link" type="gpu_lidar">
         <inertial>
@@ -28,37 +25,4 @@
           </geometry>
         </collision>
-        <sensor name='base_laser_front' type='gpu_lidar'>
-          <pose relative_to="lidar_frame">0 0 0 0 0 0</pose>
-          <update_rate>10</update_rate>
-          <topic>lidar</topic>
-          <ray>
-            <scan>
-              <horizontal>
-                  <samples>150</samples>
-                  <resolution>1</resolution>
-                  <min_angle>-1.57</min_angle>
-                  <max_angle>1.57</max_angle>
-              </horizontal>
-             <vertical>
-                  <samples>1</samples>
-                  <resolution>0.01</resolution>
-                  <min_angle>0</min_angle>
-                  <max_angle>0</max_angle>
-              </vertical>
-            </scan>
-              <range>
-                  <min>0.05</min>
-                  <max>5.6</max>
-                  <resolution>0.36</resolution>
-              </range>
-             <!-- <noise>
-                  <type>gaussian</type>
-                  <mean>0.00</mean>
-                  <stddev>0.01</stddev>
-              </noise>-->
-          </ray>
-          <always_on>1</always_on>
-          <visualize>true</visualize>
-        </sensor>
     </link>
 </robot>
