Commit message: start with robocup

File: youbot/youbot_controller/src/youbot_base_gazebo_plugins.urdf.xacro (robot description, xacro)
@@ -2,5 +2,5 @@
 <robot xmlns:xacro="http://www.ros.org/wiki/xacro" >
     <gazebo>
-      <plugin filename="libignition-gazebo-diff-drive-system.so" name="ignition::gazebo::systems::DiffDrive">
+      <plugin filename="libignition-gazebo-diff-drive-system" name="ignition::gazebo::systems::DiffDrive">
         <left_joint>wheel_joint_fl</left_joint>
         <left_joint>wheel_joint_bl</left_joint>

File: youbot/youbot_controller/src/youbot_lidar_gazebo_plugins.urdf.xacro (robot description, xacro)
@@ -3,7 +3,7 @@
   <gazebo reference="base_laser_front_link">
     <sensor name='base_laser_front' type='gpu_lidar'>
-      <pose>0 0 0 0 0 0</pose>
+      <pose relative_to="base_laser_front_link">0 0 0 0 0 0</pose>
       <update_rate>10</update_rate>
-      <visualize>true</visualize>
+      <topic>lidar</topic>
       <ray>
         <scan>
@@ -14,6 +14,7 @@
               <max_angle>1.57</max_angle>
           </horizontal>
-          <vertical>
+         <vertical>
               <samples>1</samples>
+              <resolution>0.01</resolution>
               <min_angle>0</min_angle>
               <max_angle>0</max_angle>
@@ -25,19 +26,20 @@
               <resolution>0.36</resolution>
           </range>
-          <noise>
+         <!-- <noise>
               <type>gaussian</type>
               <mean>0.00</mean>
               <stddev>0.01</stddev>
-          </noise>
+          </noise>-->
       </ray>
+      <always_on>1</always_on>
+      <visualize>true</visualize>
     </sensor>
     <plugin name='gazebo_ros_base_laser_front_controller' filename='libignition-gazebo-sensors-system.so'>
+      <output_type>sensor_msgs/LaserScan</output_type>
       <ros>
-       <!--   <argument> -  -ros-args - -remap ~/out:=scan</argument>
-      -->
-      <argument>~/out:=scan</argument>
+        <argument>~/out:=scan</argument>
       </ros>
-      <output_type>sensor_msgs/LaserScan</output_type>
-      <frame_name>/scan</frame_name>
+      <frame>lidar_frame</frame>
+      <render_engine>ogre2</render_engine>
     </plugin>
   </gazebo>

File: youbot/youbot_model_description/urdf/youbot.urdf.xacro (robot description, xacro)
@@ -2,8 +2,8 @@
 <robot xmlns:xacro="http://www.ros.org/wiki/xacro" name="youbot">
     <xacro:include filename="youbot_base.xacro" />
-    <xacro:include filename="youbot_lidar.xacro" />
     <xacro:include filename="$(find youbot_controller)/src/youbot_base_gazebo_plugins.urdf.xacro"/>
-    <xacro:include filename="$(find youbot_controller)/src/youbot_lidar_gazebo_plugins.urdf.xacro"/>
     <!--
+          <xacro:include filename="$(find youbot_controller)/src/youbot_lidar_gazebo_plugins.urdf.xacro"/>
+       <xacro:include filename="youbot_lidar.xacro" />
     <xacro:include filename="$(find youbot_controller)/src/youbot_arm_gazebo_plugins.urdf.xacro"/>
       <xacro:include filename="$(find youbot_controller)/src/ros_controller.urdf.xacro"/>

File: youbot/youbot_model_description/urdf/youbot_base.xacro (robot description, xacro)
@@ -48,10 +48,10 @@
       <parent link="base_footprint"/>
     </joint>
-    <!-- BASE_LINK-->
+   <!--  BASE_LINK-->
     <link name="base_link">
       <inertial>
-        <mass value="22.0"/>
-        <origin xyz="0 0 0"/>
-        <inertia ixx="5.652232699207" ixy="-0.009719934438" ixz="1.293988226423" iyy="5.669473158652" iyz="-0.007379583694" izz="3.683196351726"/>
+        <mass value="19.0"/>
+        <origin xyz="0 0 0"/>
+        <inertia ixx="5.652232699207" ixy="0" ixz="1.293988226423" iyy="5.669473158652" iyz="0" izz="3.683196351726"/>
       </inertial>
       <visual>
@@ -79,5 +79,5 @@
         <mass value="0.1"/>
         <origin xyz="0 0 0"/>
-        <inertia ixx="0.012411765597" ixy="-0.000711733678" ixz="0.00050272983" iyy="0.015218160428" iyz="-0.000004273467" izz="0.011763977943"/>
+        <inertia ixx="0.012411765597" ixy="0" ixz="0.00050272983" iyy="0.015218160428" iyz="0" izz="0.011763977943"/>
       </inertial>
     </link>
@@ -93,7 +93,7 @@
     <link name="wheel_link_fl">
       <inertial>
-        <mass value="0.4"/>
-        <origin xyz="0 0 0"/>
-        <inertia ixx="0.012411765597" ixy="-0.000711733678" ixz="0.00050272983" iyy="0.015218160428" iyz="-0.000004273467" izz="0.011763977943"/>
+        <mass value="1.4"/>
+        <origin xyz="0 0 0"/>
+        <inertia ixx="0.012411765597" ixy="0" ixz="0.00050272983" iyy="0.015218160428" iyz="0" izz="0.011763977943"/>
       </inertial>
       <visual>
@@ -121,5 +121,5 @@
         <mass value="0.1"/>
         <origin xyz="0 0 0"/>
-        <inertia ixx="0.012411765597" ixy="-0.000711733678" ixz="0.00050272983" iyy="0.015218160428" iyz="-0.000004273467" izz="0.011763977943"/>
+        <inertia ixx="0.012411765597" ixy="0" ixz="0.00050272983" iyy="0.015218160428" iyz="0" izz="0.011763977943"/>
       </inertial>
     </link>
@@ -135,7 +135,7 @@
     <link name="wheel_link_fr">
       <inertial>
-        <mass value="0.4"/>
-        <origin xyz="0 0 0"/>
-        <inertia ixx="0.012411765597" ixy="-0.000711733678" ixz="0.00050272983" iyy="0.015218160428" iyz="-0.000004273467" izz="0.011763977943"/>
+        <mass value="1.4"/>
+        <origin xyz="0 0 0"/>
+        <inertia ixx="0.012411765597" ixy="0" ixz="0.00050272983" iyy="0.015218160428" iyz="0" izz="0.011763977943"/>
       </inertial>
       <visual>
@@ -163,5 +163,5 @@
         <mass value="0.1"/>
         <origin xyz="0 0 0"/>
-        <inertia ixx="0.012411765597" ixy="-0.000711733678" ixz="0.00050272983" iyy="0.015218160428" iyz="-0.000004273467" izz="0.011763977943"/>
+        <inertia ixx="0.012411765597" ixy="0.000711733678" ixz="0.00050272983" iyy="0.015218160428" iyz="0.000004273467" izz="0.011763977943"/>
       </inertial>
     </link>
@@ -177,7 +177,7 @@
     <link name="wheel_link_bl">
       <inertial>
-        <mass value="0.4"/>
-        <origin xyz="0 0 0"/>
-        <inertia ixx="0.012411765597" ixy="-0.000711733678" ixz="0.00050272983" iyy="0.015218160428" iyz="-0.000004273467" izz="0.011763977943"/>
+        <mass value="1.4"/>
+        <origin xyz="0 0 0"/>
+        <inertia ixx="0.012411765597" ixy="0.000711733678" ixz="0.00050272983" iyy="0.015218160428" iyz="0.000004273467" izz="0.011763977943"/>
       </inertial>
       <visual>
@@ -205,5 +205,5 @@
         <mass value="0.1"/>
         <origin xyz="0 0 0"/>
-        <inertia ixx="0.012411765597" ixy="-0.000711733678" ixz="0.00050272983" iyy="0.015218160428" iyz="-0.000004273467" izz="0.011763977943"/>
+        <inertia ixx="0.012411765597" ixy="0.000711733678" ixz="0.00050272983" iyy="0.015218160428" iyz="0.000004273467" izz="0.011763977943"/>
       </inertial>
     </link>
@@ -219,7 +219,7 @@
     <link name="wheel_link_br">
       <inertial>
-        <mass value="0.4"/>
-        <origin xyz="0 0 0"/>
-        <inertia ixx="0.012411765597" ixy="-0.000711733678" ixz="0.00050272983" iyy="0.015218160428" iyz="-0.000004273467" izz="0.011763977943"/>
+        <mass value="1.4"/>
+        <origin xyz="0 0 0"/>
+        <inertia ixx="0.012411765597" ixy="0.000711733678" ixz="0.00050272983" iyy="0.015218160428" iyz="0.000004273467" izz="0.011763977943"/>
       </inertial>
       <visual>

Commit message: change world file

File: youbot/youbot_controller/src/youbot_base_gazebo_plugins.urdf.xacro (robot description, xacro)
@@ -2,5 +2,5 @@
 <robot xmlns:xacro="http://www.ros.org/wiki/xacro" >
     <gazebo>
-      <plugin filename="libignition-gazebo-diff-drive-system" name="ignition::gazebo::systems::DiffDrive">
+      <plugin filename="libignition-gazebo-diff-drive-system.so" name="ignition::gazebo::systems::DiffDrive">
         <left_joint>wheel_joint_fl</left_joint>
         <left_joint>wheel_joint_bl</left_joint>
@@ -22,4 +22,11 @@
       </plugin>
       <!--
+             <plugin name="omni_steering" filename="libgazebo_ros_planar_move.so">
+        <commandTopic>cmd_vel</commandTopic>
+        <odometryTopic>odom</odometryTopic>
+        <odometryRate>10</odometryRate>
+        <robotBaseFrame>base_footprint</robotBaseFrame>
+        <publishTF>true</publishTF>
+      </plugin>
         <plugin name='base_controller'
               filename='libgazebo_ros_planar_move.so'>
@@ -49,11 +56,4 @@
         <mu2 value ="0.001"/>
       </gazebo>
-      <plugin name="omni_steering" filename="libgazebo_ros_planar_move.so">
-        <commandTopic>cmd_vel</commandTopic>
-        <odometryTopic>odom</odometryTopic>
-        <odometryRate>10</odometryRate>
-        <robotBaseFrame>base_footprint</robotBaseFrame>
-        <publishTF>true</publishTF>
-      </plugin>
     <plugin name="skid_steer_drive_controller" filename="libgazebo_ros_skid_steer_drive.so">
         <topic>cmd_vel</topic>

File: youbot/youbot_gazebo/worlds/robocup_at_work_2012.urdf (robot description, URDF)
Before this commit: robot arena, 10 links, 0 joints
Joints:
- added joint join1: type fixed, parent wall_1, child wall_2, origin xyz=2 0 0 rpy=0 0 0
- added joint join10: type fixed, parent wall_2, child wall_10, origin xyz=-0.25 0.0 0.0 rpy=0 0 0
- added joint join2: type fixed, parent wall_2, child wall_3, origin xyz=-2 -1.2 0 rpy=0 0 0
- added joint join3: type fixed, parent wall_3, child wall_4, origin xyz=0 -0.4 0 rpy=0 0 0
- added joint join4: type fixed, parent wall_1, child wall_5, origin xyz=0 0 0 rpy=0 0 0
- added joint join5: type fixed, parent wall_3, child wall_6, origin xyz=-2 -0.4 0 rpy=0 0 0
- added joint join6: type fixed, parent wall_1, child wall_7, origin xyz=-2 0 0 rpy=0 0 0
- added joint join7: type fixed, parent wall_7, child wall_8, origin xyz=0.25 0.8 0.0 rpy=0 0 0
- added joint join8: type fixed, parent wall_6, child wall_9, origin xyz=0.25 0.8 0.0 rpy=0 0 0

File: youbot/youbot_model_description/urdf/youbot.urdf.xacro (robot description, xacro)
@@ -2,8 +2,9 @@
 <robot xmlns:xacro="http://www.ros.org/wiki/xacro" name="youbot">
     <xacro:include filename="youbot_base.xacro" />
+    xacro:include filename="$(find youbot_controller)/src/youbot_lidar_gazebo_plugins.urdf.xacro"/>
+    <xacro:include filename="youbot_lidar.xacro" />
     <xacro:include filename="$(find youbot_controller)/src/youbot_base_gazebo_plugins.urdf.xacro"/>
     <!--
-          <xacro:include filename="$(find youbot_controller)/src/youbot_lidar_gazebo_plugins.urdf.xacro"/>
-       <xacro:include filename="youbot_lidar.xacro" />
+          <
     <xacro:include filename="$(find youbot_controller)/src/youbot_arm_gazebo_plugins.urdf.xacro"/>
       <xacro:include filename="$(find youbot_controller)/src/ros_controller.urdf.xacro"/>
