Commit message: robocup at work delete joints

File: youbot/youbot_gazebo/worlds/robocup_at_work_2012.urdf (robot description, URDF)
Before this commit: robot arena, 10 links, 9 joints
Joints:
- removed joint join1
- removed joint join10
- removed joint join2
- removed joint join3
- removed joint join4
- removed joint join5
- removed joint join6
- removed joint join7
- removed joint join8
